File: examples/stm32/l0/l0x2/stm32l052k8t/usb_speaker/hardware/usb_speaker.sch (EAGLE design)
At the start: 40 parts, among them IC1 LM4040D20IDBZ, IC2 LMV358M, IC3 MCP4822-E/SN, IC4 DS1881E, IC5 LM4861M, IC6 LM4861M, M1 STM32L052K8T_DIP, X1 MKDSN1,5/2-5,08, X2 MKDSN1,5/2-5,08, X3 MINI-USB-UX60A-MB-5ST

Commit message: Fix usb_speaker.
Parts:
- added R12, R14: 20k, resistor:R-EU_0207/2V
- added R13, R15: 20k, resistor:R-EU_0207/10
- R10: value 20k -> 4.7k
- R11: value 20k -> 4.7k; device resistor:R-EU_0207/10 -> resistor:R-EU_0207/2V
- R3, R4: value 180 -> 20.0k
- R5: value 10k -> 180
- R6: value 22 -> 180; device resistor:R-EU_0207/10 -> resistor:R-EU_0207/2V
- R7: value 22 -> 10k; device resistor:R-EU_0207/10 -> resistor:R-EU_0207/2V
- R8: value 20k -> 22; device resistor:R-EU_0207/2V -> resistor:R-EU_0207/10
- R9: value 20k -> 22
Connections:
- new net N$14: C2.1, IC1.C, R2.1, R3.1
- net +3V3: now also C4.1, C5.1, IC3.VDD, R10.2, R11.2, R6.2, R7.2; no longer R3.2, R4.2
- net +5V: no longer C4.1, C5.1, IC3.VDD
- net GND: now also R4.1
- net N$10: now also R7.1; no longer R5.1
- net N$16: now also R12.2, R13.1; no longer R8.2, R9.1
- net N$17: now also R12.1; no longer R8.1
- net N$20: now also R13.2; no longer R9.2
- net N$22: now also R14.1; no longer R10.1
- net N$23: now also R14.2, R15.1; no longer R10.2, R11.1
- net N$25: now also R15.2; no longer R11.2
- net N$30: now also R9.1; no longer R7.1
- net N$31: now also R8.1; no longer R6.1
- net N$33: now also R9.2; no longer R7.2
- net N$35: now also R8.2; no longer R6.2
- net N$38: now also R10.1
- net N$39: now also R3.2, R4.2; no longer C2.1, IC1.C, R2.1
- net N$41: now also R11.1
- net N$7: now also R6.1; no longer R4.1
- net N$9: now also R5.1; no longer R3.1
Other:
- moved on the sheet: C2, IC1, R10, R11, R2, R3, R4, R5, R6, R7, R8, R9
