File: examples/stm32/l0/l0x2/stm32l052k8t/button/hardware/button.sch (EAGLE design)
At the start: 12 parts, among them M1 STM32L052K8T_DIP

Commit message: Fix button.
Parts:
- S1: value SWITCH-MOMENTARY-212MM -> SKRGAAD010; device SparkFun-Electromechanical:SWITCH-MOMENTARY-212MM -> switch-alps:SKRGAAD010
Changed lines of the file:
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@@
 <?xml version="1.0" encoding="utf-8"?>
 <!DOCTYPE eagle SYSTEM "eagle.dtd">
-<eagle version="7.5.0">
+<eagle version="8.2.2">
 <drawing>
 <settings>
@@
 <setting verticaltext="up"/>
 </settings>
-<grid distance="0.1" unitdist="inch" unit="inch" style="lines" multiple="1" display="yes" altdistance="0.01" altunitdist="inch" altunit="inch"/>
+<grid distance="0.1" unitdist="inch" unit="inch" style="lines" multiple="1" display="no" altdistance="0.01" altunitdist="inch" altunit="inch"/>
 <layers>
 <layer number="1" name="Top" color="4" fill="1" visible="no" active="no"/>
@@
 <part name="R5" library="resistor" deviceset="R-EU_" device="0207/2V" value="100"/>
 <part name="C2" library="cap" deviceset="C-JIS" device="050-024X044" value="1uF"/>
-<part name="S1" library="SparkFun-Electromechanical" deviceset="SWITCH-MOMENTARY-2" device="12MM"/>
 <part name="+3V5" library="supply1" deviceset="+3V3" device=""/>
 <part name="GND2" library="supply1" deviceset="GND" device=""/>
 <part name="GND7" library="supply1" deviceset="GND" device=""/>
+<part name="S1" library="switch-alps" deviceset="SKRG" device="" technology="AAD010"/>
 </parts>
 <sheets>
@@
 <instance part="R5" gate="G$1" x="104.14" y="2.54"/>
 <instance part="C2" gate="G$1" x="96.52" y="-2.54"/>
-<instance part="S1" gate="G$1" x="81.28" y="-5.08" smashed="yes" rot="R90">
-<attribute name="NAME" x="78.74" y="-7.62" size="1.778" layer="95" rot="R90"/>
-<attribute name="VALUE" x="73.66" y="-7.62" size="1.778" layer="96" rot="R90"/>
-</instance>
 <instance part="+3V5" gate="G$1" x="81.28" y="20.32"/>
 <instance part="GND2" gate="1" x="96.52" y="-15.24"/>
 <instance part="GND7" gate="1" x="81.28" y="-15.24"/>
+<instance part="S1" gate="G$1" x="81.28" y="-5.08" smashed="yes">
+<attribute name="NAME" x="74.93" y="-7.62" size="1.778" layer="95" rot="R90"/>
+<attribute name="VALUE" x="73.66" y="0" size="1.778" layer="96" rot="R90"/>
+</instance>
 </instances>
 <busses>
@@
 </segment>
 <segment>
-<pinref part="S1" gate="G$1" pin="1"/>
 <pinref part="GND7" gate="1" pin="GND"/>
 <wire x1="81.28" y1="-10.16" x2="81.28" y2="-12.7" width="0.1524" layer="91"/>
+<pinref part="S1" gate="G$1" pin="1"/>
 </segment>
 <segment>
@@
 <segment>
 <pinref part="R3" gate="G$1" pin="1"/>
-<pinref part="S1" gate="G$1" pin="2"/>
 <wire x1="81.28" y1="5.08" x2="81.28" y2="2.54" width="0.1524" layer="91"/>
 <pinref part="R4" gate="G$1" pin="1"/>
@@
 <wire x1="81.28" y1="2.54" x2="83.82" y2="2.54" width="0.1524" layer="91"/>
 <junction x="81.28" y="2.54"/>
-</segment>
-</net>
+<pinref part="S1" gate="G$1" pin="2"/>
+</segment>
+</net>
