File: examples/stm32/l0/l0x2/stm32l052k8t/kitchen_timer/hardware/kitchen_timer.sch (EAGLE design)
At the start: 20 parts, among them IC1 MAX1724EZK30, M1 STM32L052K8T_DIP, M2 AQM1248_MODULE, M3 5-WAY_TACT_SW-BREAKOUT

Commit message: Fix kitchen_timer.
Parts:
- removed M3: 5-WAY_TACT_SW-BREAKOUT, sparkfun:5-WAY_TACT_SW-BREAKOUT
- added R10, R6, R7, R8, R9: 10k, resistor:R-EU_0207/7
- added S2, S3, S4, S5, S6: SKRGALD010, switch-alps:SKRGALD010
- S1: value (none) -> SKRGAAD010; device switch-omron:10-XX -> switch-alps:SKRGAAD010
Connections:
- net GND: now also S1.1, S2.1, S3.1, S4.1, S5.1, S6.1; no longer M3.-, S1.P
- net N$17: now also R6.1, S3.2; no longer M3.R
- net N$18: now also R7.1, S2.2; no longer M3.D
- net N$19: now also R8.1, S4.2; no longer M3.L
- net N$20: now also M1.PB7, R10.1, S5.2; no longer M1.PB6, M3.C
- net N$21: now also M1.PB6, R9.1, S6.2; no longer M1.PB7, M3.U
- net N$4: now also S1.2; no longer S1.S
- net VDD: now also R10.2, R6.2, R7.2, R8.2, R9.2; no longer M3.+
Other:
- note added: "3.0 V"
- note added: "Down"
- note added: "Enter"
- note added: "Left"
- note added: "Reset"
- note added: "Right"
- note added: "Up"
- moved on the sheet: BATT1, C1, C2, C3, C4, C5, IC1, JP1, L1, M1, M2, R1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
